File: PistolsFiring/PistolsFiring_KiCAD_MrKeebs/PistolsFiring_KLE.kicad_pcb (KiCad board)
At the start: 2 copper layers, 444.1 x 129.8 mm, 231 parts, among them SW1 SW_PUSH, U3 ATMEGA32U4, X3 XTAL_GND

Commit message: PistolsFiring Update
Quick idea from scratch. Probably won't be updated beyond this state for a while.
Parts:
- removed C15, C16, C17, C18, C19, C20, C21: 22pF, Capacitor_SMD:C_0805_2012Metric_Pad1.15x1.40mm_HandSolder
- removed D_11, D_12, D_13, D_14: D, keyboard_parts:D_SOD123_axial
- removed the K_ at (381.9, 29.5)
- removed K_11, K_12, K_13: KEYSW, MX_Alps_Hybrid:MX-1U-NoLED
- removed K_14: KEYSW, MX_Alps_Hybrid:MX-6.25U-NoLED
- removed R10, R9: 10k, Resistor_SMD:R_0805_2012Metric_Pad1.15x1.40mm_HandSolder
- removed R11, R12: 22u, Resistor_SMD:R_0805_2012Metric_Pad1.15x1.40mm_HandSolder
- removed U3: ATMEGA32U4, Package_QFP:TQFP-44_10x10mm_P0.8mm
- removed USB3: USB_mini_micro_B, keyboard_parts:USB_miniB_hirose_5S8
- removed X3: XTAL_GND, Crystal:Crystal_SMD_5032-4Pin_5.0x3.2mm
- added C10: 22pF, Capacitor_SMD:C_0805_2012Metric_Pad1.15x1.40mm_HandSolder, B.Cu at (463.1, 25.0)
- added C11: 22pF, Capacitor_SMD:C_0805_2012Metric_Pad1.15x1.40mm_HandSolder, B.Cu at (463.1, 50.0)
- added C12: 22pF, Capacitor_SMD:C_0805_2012Metric_Pad1.15x1.40mm_HandSolder, B.Cu at (468.1, 50.0)
- added C13: 22pF, Capacitor_SMD:C_0805_2012Metric_Pad1.15x1.40mm_HandSolder, B.Cu at (473.1, 50.0)
- added C14: 22pF, Capacitor_SMD:C_0805_2012Metric_Pad1.15x1.40mm_HandSolder, B.Cu at (478.1, 50.0)
- added C8: 22pF, Capacitor_SMD:C_0805_2012Metric_Pad1.15x1.40mm_HandSolder, B.Cu at (463.1, 40.0)
- added C9: 22pF, Capacitor_SMD:C_0805_2012Metric_Pad1.15x1.40mm_HandSolder, B.Cu at (473.1, 40.0)
- added D_LEDTOG: D, keyboard_parts:D_SOD123_axial, F.Cu at (372.9, 30.0)
- added D_NEXT: D, keyboard_parts:D_SOD123_axial, F.Cu at (430.1, 30.0)
- added D_PLAY/PAUSE: D, keyboard_parts:D_SOD123_axial, F.Cu at (411.0, 30.0)
- added D_PREV: D, keyboard_parts:D_SOD123_axial, F.Cu at (392.0, 30.0)
- added K_: KEYSW, MX_Alps_Hybrid:MX-6.25U-NoLED, F.Cu at (151.0, 134.3)
- added K_LEDTOG: KEYSW, MX_Alps_Hybrid:MX-1U-NoLED, F.Cu at (381.9, 29.5)
- added K_NEXT: KEYSW, MX_Alps_Hybrid:MX-1U-NoLED, F.Cu at (439.1, 29.5)
- added K_PLAY/PAUSE: KEYSW, MX_Alps_Hybrid:MX-1U-NoLED, F.Cu at (420.1, 29.5)
- added K_PREV: KEYSW, MX_Alps_Hybrid:MX-1U-NoLED, F.Cu at (401.0, 29.5)
- added R5: 10k, Resistor_SMD:R_0805_2012Metric_Pad1.15x1.40mm_HandSolder, B.Cu at (472.1, 15.0)
- added R6: 10k, Resistor_SMD:R_0805_2012Metric_Pad1.15x1.40mm_HandSolder, B.Cu at (483.1, 28.0)
- added R7: 22u, Resistor_SMD:R_0805_2012Metric_Pad1.15x1.40mm_HandSolder, B.Cu at (463.1, 28.0)
- added R8: 22u, Resistor_SMD:R_0805_2012Metric_Pad1.15x1.40mm_HandSolder, B.Cu at (463.1, 32.0)
- added U2: ATMEGA32U4, Package_QFP:TQFP-44_10x10mm_P0.8mm, B.Cu at (472.1, 25.0)
- added USB2: USB_mini_micro_B, keyboard_parts:USB_miniB_hirose_5S8, B.Cu at (239.1, 25.0)
- added X2: XTAL_GND, Crystal:Crystal_SMD_5032-4Pin_5.0x3.2mm, B.Cu at (468.1, 40.0)
- moved D_1 353.6 mm to (39.5, 58.6)
- moved K_1 353.6 mm to (48.6, 58.1)
- moved K_2 353.6 mm to (67.6, 58.1)
- moved K_3 353.6 mm to (86.7, 58.1)
- moved D_2 353.6 mm to (58.6, 58.6)
- moved D_3 353.6 mm to (77.7, 58.6)
- moved D_ 299.9 mm to (91.9, 134.8)
- moved D_10 241.2 mm to (392.0, 96.7)
- moved K_10 241.2 mm to (401.0, 96.2)
- moved D_4 57.2 mm to (96.7, 58.6)
- moved D_6 57.2 mm to (134.8, 58.6)
- moved D_8 57.2 mm to (172.9, 58.6)
- moved K_5 57.2 mm to (124.8, 58.1)
- moved K_7 57.2 mm to (162.9, 58.1)
- moved K_8 57.2 mm to (181.9, 58.1)
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Connections:
- D_ pad 1: /col16 -> /col3
- D_1 pad 1: /col17 -> /col1
- D_10 pad 1: /col7 -> /col14
- D_2 pad 1: /col18 -> /col2
- D_3 pad 1: /col19 -> /col3
- D_4 pad 1: /col1 -> /col4
- D_5 pad 1: /col2 -> /col5
- D_6 pad 1: /col3 -> /col6
- D_7 pad 1: /col4 -> /col7
- D_8 pad 1: /col5 -> /col8
- D_9 pad 1: /col6 -> /col9
